File: kicad/parasite.kicad_pcb (KiCad board)
At the start: 2 copper layers, 22 x 300 mm, 42 parts, among them J1 JLINK-6PIN, U1 E73-2G4M08S1C-52840, U2 BQ25504, Y1 32.768kHz

Commit message: Cleared remaining DRC, add JLCPCB part numbers
Parts:
- R5: value 5.23 -> 4.99M
- U1: footprint nrfmicro:E73-2G4M08S1C-52840 -> solar-bug:E73-2G4M08S1C-52840
- moved R12 2.00 mm to (72.4, 100.8), turned to -90 degrees
- moved R10 1.00 mm to (73.4, 100.8)
- moved R11 1.00 mm to (74.4, 100.9)
- moved TP4 0.11 mm to (79.4, 97.2)
Connections:
- R11 pad 2: Net-(R11-Pad2) -> GND
- R12 pad 1: Net-(R11-Pad2) -> Net-(R12-Pad1)
- R9 pad 2: GND -> Net-(R12-Pad1)
Routing:
- net Net-(R12-Pad1): track 0.00 -> 1.44 mm
- net GND: track 489.4 -> 488.3 mm
- net Net-(R11-Pad2): track 1.00 -> 0.00 mm
- net /VBAT_OK: track 12.9 -> 13.8 mm
- net /VBAT: vias 2 -> 1
- removed copper zone on F.Cu, net +3V0
Other:
- board text added: "(1) Solder solar cell perpendicular to the board"
- board text added: "ASSEMBLY NOTES:"
