File: kicad/solar-bug/solar-bug.kicad_sch (KiCad schematic)
At the start: 42 parts, among them J1 JLINK-6PIN, U1 E73-2G4M08S1C-52840, U2 BQ25504, Y1 32.768kHz

Commit message: clean-up folder, renamed project file
Parts:
- C1: LCSC (none) -> C15195
- C2, C5, C6: LCSC (none) -> C23733
- C3, C4: LCSC (none) -> C1547
- D1: LCSC (none) -> C160479
- L1: LCSC (none) -> C2880384
- R1, R2, R9: LCSC (none) -> C477747
- R10, R11, R4, R5, R7: LCSC (none) -> C137963
- R12, R13, R14, R15: LCSC (none) -> C26083
- R3, R6: LCSC (none) -> C163464
- R8: LCSC (none) -> C11702
- U1: LCSC (none) -> C356849
- U2: LCSC (none) -> C157471
- Y1: LCSC (none) -> C398713
Changed lines of the file:
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@@
       (effects (font (size 1.27 1.27)) hide)
     )
-    (property "LCSC" "" (id 4) (at 266.7 91.44 90)
+    (property "LCSC" "C11702" (id 4) (at 266.7 91.44 90)
       (effects (font (size 1.27 1.27)) hide)
     )
@@
       (effects (font (size 1.27 1.27)) hide)
     )
-    (property "LCSC" "" (id 4) (at 254 91.44 0)
+    (property "LCSC" "C160479" (id 4) (at 254 91.44 0)
       (effects (font (size 1.27 1.27)) hide)
     )
@@
       (effects (font (size 1.27 1.27)) hide)
     )
-    (property "LCSC" "" (id 4) (at 254 69.85 90)
+    (property "LCSC" "C398713" (id 4) (at 254 69.85 90)
       (effects (font (size 1.27 1.27)) hide)
     )
@@
       (effects (font (size 1.27 1.27)) hide)
     )
-    (property "LCSC" "" (id 4) (at 266.7 73.66 0)
+    (property "LCSC" "C1547" (id 4) (at 266.7 73.66 0)
       (effects (font (size 1.27 1.27)) hide)
     )
@@
       (effects (font (size 1.27 1.27)) hide)
     )
-    (property "LCSC" "" (id 4) (at 266.7 66.04 0)
+    (property "LCSC" "C1547" (id 4) (at 266.7 66.04 0)
       (effects (font (size 1.27 1.27)) hide)
     )
@@
       (effects (font (size 1.27 1.27)) hide)
     )
-    (property "LCSC" "" (id 4) (at 63.5 101.6 0)
+    (property "LCSC" "C137963" (id 4) (at 63.5 101.6 0)
       (effects (font (size 1.27 1.27)) hide)
     )
@@
       (effects (font (size 1.27 1.27)) hide)
     )
-    (property "LCSC" "" (id 4) (at 208.28 45.72 0)
+    (property "LCSC" "C356849" (id 4) (at 208.28 45.72 0)
       (effects (font (size 1.27 1.27)) hide)
     )
@@
       (effects (font (size 1.27 1.27)) hide)
     )
-    (property "LCSC" "" (id 4) (at 58.42 78.74 0)
+    (property "LCSC" "C477747" (id 4) (at 58.42 78.74 0)
       (effects (font (size 1.27 1.27)) hide)
     )
@@
     )
     (property "MPN" "NR4018T220M" (id 4) (at 96.52 60.96 90))
-    (property "LCSC" "" (id 5) (at 91.44 63.5 0)
+    (property "LCSC" "C2880384" (id 5) (at 91.44 63.5 0)
       (effects (font (size 1.27 1.27)) hide)
     )
@@
       (effects (font (size 1.27 1.27)) hide)
     )
-    (property "LCSC" "" (id 4) (at 76.2 106.68 0)
+    (property "LCSC" "C15195" (id 4) (at 76.2 106.68 0)
       (effects (font (size 1.27 1.27)) hide)
     )
@@
       (effects (font (size 1.27 1.27)) hide)
     )
-    (property "LCSC" "" (id 4) (at 53.34 101.6 0)
+    (property "LCSC" "C477747" (id 4) (at 53.34 101.6 0)
       (effects (font (size 1.27 1.27)) hide)
     )
@@
       (effects (font (size 1.27 1.27)) hide)
     )
-    (property "LCSC" "" (id 4) (at 58.42 68.58 0)
+    (property "LCSC" "C163464" (id 4) (at 58.42 68.58 0)
       (effects (font (size 1.27 1.27)) hide)
     )
@@
       (effects (font (size 1.27 1.27)) hide)
     )
-    (property "LCSC" "" (id 4) (at 44.45 106.68 0)
+    (property "LCSC" "C137963" (id 4) (at 44.45 106.68 0)
       (effects (font (size 1.27 1.27)) hide)
     )
@@
       (effects (font (size 1.27 1.27)) hide)
     )
-    (property "LCSC" "" (id 4) (at 180.34 71.12 0)
+    (property "LCSC" "C23733" (id 4) (at 180.34 71.12 0)
       (effects (font (size 1.27 1.27)) hide)
     )
@@
       (effects (font (size 1.27 1.27)) hide)
     )
-    (property "LCSC" "" (id 4) (at 111.76 114.3 0)
+    (property "LCSC" "C157471" (id 4) (at 111.76 114.3 0)
       (effects (font (size 1.27 1.27)) hide)
     )
@@
       (effects (font (size 1.27 1.27)) hide)
     )
-    (property "LCSC" "" (id 4) (at 266.7 99.06 0)
+    (property "LCSC" "C26083" (id 4) (at 266.7 99.06 0)
       (effects (font (size 1.27 1.27)) hide)
     )
@@
       (effects (font (size 1.27 1.27)) hide)
     )
-    (property "LCSC" "" (id 4) (at 266.7 101.6 0)
+    (property "LCSC" "C26083" (id 4) (at 266.7 101.6 0)
       (effects (font (size 1.27 1.27)) hide)
     )
@@
       (effects (font (size 1.27 1.27)) hide)
     )
-    (property "LCSC" "" (id 4) (at 33.02 96.52 0)
+    (property "LCSC" "C163464" (id 4) (at 33.02 96.52 0)
       (effects (font (size 1.27 1.27)) hide)
     )
@@
       (effects (font (size 1.27 1.27)) hide)
     )
-    (property "LCSC" "" (id 4) (at 33.02 93.98 0)
+    (property "LCSC" "C137963" (id 4) (at 33.02 93.98 0)
       (effects (font (size 1.27 1.27)) hide)
     )
@@
       (effects (font (size 1.27 1.27)) hide)
     )
-    (property "LCSC" "" (id 4) (at 53.34 111.76 0)
+    (property "LCSC" "C26083" (id 4) (at 53.34 111.76 0)
       (effects (font (size 1.27 1.27)) hide)
     )
@@
       (effects (font (size 1.27 1.27)) hide)
     )
-    (property "LCSC" "" (id 4) (at 266.7 104.14 0)
+    (property "LCSC" "C26083" (id 4) (at 266.7 104.14 0)
       (effects (font (size 1.27 1.27)) hide)
     )
@@
       (effects (font (size 1.27 1.27)) hide)
     )
-    (property "LCSC" "" (id 4) (at 76.2 71.12 0)
+    (property "LCSC" "C23733" (id 4) (at 76.2 71.12 0)
       (effects (font (size 1.27 1.27)) hide)
     )
@@
       (effects (font (size 1.27 1.27)) hide)
     )
-    (property "LCSC" "" (id 4) (at 33.02 91.44 0)
+    (property "LCSC" "C137963" (id 4) (at 33.02 91.44 0)
       (effects (font (size 1.27 1.27)) hide)
     )
@@
       (effects (font (size 1.27 1.27)) hide)
     )
-    (property "LCSC" "" (id 4) (at 58.42 73.66 0)
+    (property "LCSC" "C477747" (id 4) (at 58.42 73.66 0)
       (effects (font (size 1.27 1.27)) hide)
     )
@@
       (effects (font (size 1.27 1.27)) hide)
     )
-    (property "LCSC" "" (id 4) (at 63.5 111.76 0)
+    (property "LCSC" "C137963" (id 4) (at 63.5 111.76 0)
       (effects (font (size 1.27 1.27)) hide)
     )
@@
       (effects (font (size 1.27 1.27)) hide)
     )
-    (property "LCSC" "" (id 4) (at 119.38 106.68 0)
-      (effects (font (size 1.27 1.27)) hide)
-    )
+    (property "LCSC" "C23733" (id 4) (at 119.38 106.68 0)
+      (effects (font (size 1.27 1.27)) hide)
+    )

Commit message: Add Digikey PNs to BOM, generate BOM CSV
Parts:
- C1: DK (none) -> 490-GRM1555CYA103GE01DCT-ND
- C2, C5, C6: DK (none) -> 490-GRM155D81C475ME15JCT-ND
- C3, C4: DK (none) -> 490-GRT1555C1E120JA02JCT-ND
- D1: DK (none) -> 754-1811-1-ND
- L1: DK (none) -> 587-2889-1-ND
- R1, R2, R9: DK (none) -> 541-5.23MLCT-ND
- R10, R11, R4, R5, R7: DK (none) -> 13-RC0402FR-074M99LCT-ND
- R12, R13, R14, R15: DK (none) -> 311-1.00MLRCT-ND
- R3, R6: DK (none) -> 13-RC0402FR-073M01LCT-ND
- R8: DK (none) -> 311-1.00KLRCT-ND
- U2: DK (none) -> 296-29741-1-ND
- Y1: DK (none) -> 535-11899-1-ND
Changed lines of the file:
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@@
+      (effects (font (size 1.27 1.27)) hide)
+    )
+    (property "DK" "311-1.00KLRCT-ND" (id 7) (at 266.7 91.44 0)
       (effects (font (size 1.27 1.27)) hide)
     )
@@
       (effects (font (size 1.27 1.27)) hide)
     )
+    (property "DK" "754-1811-1-ND" (id 6) (at 254 91.44 0)
+      (effects (font (size 1.27 1.27)) hide)
+    )
     (pin "1")
     (pin "2")
@@
       (effects (font (size 1.27 1.27)) hide)
     )
+    (property "DK" "535-11899-1-ND" (id 5) (at 254 69.85 0)
+      (effects (font (size 1.27 1.27)) hide)
+    )
     (pin "1")
     (pin "2")
@@
       (effects (font (size 1.27 1.27)) hide)
     )
+    (property "DK" "490-GRT1555C1E120JA02JCT-ND" (id 6) (at 266.7 73.66 0)
+      (effects (font (size 1.27 1.27)) hide)
+    )
     (pin "1")
     (pin "2")
@@
     )
     (property "Tolerance" "x5R" (id 5) (at 266.7 66.04 0)
+      (effects (font (size 1.27 1.27)) hide)
+    )
+    (property "DK" "490-GRT1555C1E120JA02JCT-ND" (id 6) (at 266.7 66.04 0)
       (effects (font (size 1.27 1.27)) hide)
     )
@@
     )
     (property "Tolerance" "1%" (id 6) (at 63.5 101.6 0)
+      (effects (font (size 1.27 1.27)) hide)
+    )
+    (property "DK" "13-RC0402FR-074M99LCT-ND" (id 7) (at 63.5 101.6 0)
       (effects (font (size 1.27 1.27)) hide)
     )
@@
       (effects (font (size 1.27 1.27)) hide)
     )
+    (property "DK" "541-5.23MLCT-ND" (id 7) (at 58.42 78.74 0)
+      (effects (font (size 1.27 1.27)) hide)
+    )
     (pin "1")
     (pin "2")
@@
       (effects (font (size 1.27 1.27)) hide)
     )
+    (property "DK" "587-2889-1-ND" (id 6) (at 95.25 66.04 0)
+      (effects (font (size 1.27 1.27)) hide)
+    )
     (pin "1")
     (pin "2")
@@
     (property "Tolerance" "C0G" (id 6) (at 78.74 113.03 0)
       (effects (font (size 1.27 1.27)) (justify left))
+    )
+    (property "DK" "490-GRM1555CYA103GE01DCT-ND" (id 7) (at 76.2 106.68 0)
+      (effects (font (size 1.27 1.27)) hide)
     )
     (pin "1")
@@
       (effects (font (size 1.27 1.27)) hide)
     )
+    (property "DK" "541-5.23MLCT-ND" (id 7) (at 53.34 101.6 0)
+      (effects (font (size 1.27 1.27)) hide)
+    )
     (pin "1")
     (pin "2")
@@
       (effects (font (size 1.27 1.27)) hide)
     )
+    (property "DK" "13-RC0402FR-073M01LCT-ND" (id 7) (at 58.42 68.58 0)
+      (effects (font (size 1.27 1.27)) hide)
+    )
     (pin "1")
     (pin "2")
@@
       (effects (font (size 1.27 1.27)) hide)
     )
+    (property "DK" "13-RC0402FR-074M99LCT-ND" (id 7) (at 44.45 106.68 0)
+      (effects (font (size 1.27 1.27)) hide)
+    )
     (pin "1")
     (pin "2")
@@
     )
     (property "Tolerance" "x5R" (id 6) (at 180.34 71.12 0)
+      (effects (font (size 1.27 1.27)) hide)
+    )
+    (property "DK" "490-GRM155D81C475ME15JCT-ND" (id 7) (at 180.34 71.12 0)
       (effects (font (size 1.27 1.27)) hide)
     )
@@
     )
     (property "LCSC" "C157471" (id 4) (at 111.76 114.3 0)
+      (effects (font (size 1.27 1.27)) hide)
+    )
+    (property "DK" "296-29741-1-ND" (id 5) (at 99.06 93.98 0)
       (effects (font (size 1.27 1.27)) hide)
     )
@@
       (effects (font (size 1.27 1.27)) hide)
     )
+    (property "DK" "311-1.00MLRCT-ND" (id 7) (at 266.7 99.06 0)
+      (effects (font (size 1.27 1.27)) hide)
+    )
     (pin "1")
     (pin "2")
@@
     )
     (property "Tolerance" "1%" (id 6) (at 266.7 101.6 0)
+      (effects (font (size 1.27 1.27)) hide)
+    )
+    (property "DK" "311-1.00MLRCT-ND" (id 7) (at 266.7 101.6 0)
       (effects (font (size 1.27 1.27)) hide)
     )
@@
       (effects (font (size 1.27 1.27)) hide)
     )
+    (property "DK" "13-RC0402FR-073M01LCT-ND" (id 7) (at 33.02 96.52 0)
+      (effects (font (size 1.27 1.27)) hide)
+    )
     (pin "1")
     (pin "2")
@@
     )
     (property "Tolerance" "1%" (id 6) (at 33.02 93.98 0)
+      (effects (font (size 1.27 1.27)) hide)
+    )
+    (property "DK" "13-RC0402FR-074M99LCT-ND" (id 7) (at 33.02 93.98 0)
       (effects (font (size 1.27 1.27)) hide)
     )
@@
       (effects (font (size 1.27 1.27)) hide)
     )
+    (property "DK" "311-1.00MLRCT-ND" (id 7) (at 53.34 111.76 0)
+      (effects (font (size 1.27 1.27)) hide)
+    )
     (pin "1")
     (pin "2")
@@
       (effects (font (size 1.27 1.27)) hide)
     )
+    (property "DK" "311-1.00MLRCT-ND" (id 7) (at 266.7 104.14 0)
+      (effects (font (size 1.27 1.27)) hide)
+    )
     (pin "1")
     (pin "2")
@@
     )
     (property "Tolerance" "x5R" (id 6) (at 76.2 71.12 0)
+      (effects (font (size 1.27 1.27)) hide)
+    )
+    (property "DK" "490-GRM155D81C475ME15JCT-ND" (id 7) (at 76.2 71.12 0)
       (effects (font (size 1.27 1.27)) hide)
     )
@@
       (effects (font (size 1.27 1.27)) hide)
     )
+    (property "DK" "13-RC0402FR-074M99LCT-ND" (id 7) (at 33.02 91.44 0)
+      (effects (font (size 1.27 1.27)) hide)
+    )
     (pin "1")
     (pin "2")
@@
       (effects (font (size 1.27 1.27)) hide)
     )
+    (property "DK" "541-5.23MLCT-ND" (id 7) (at 58.42 73.66 0)
+      (effects (font (size 1.27 1.27)) hide)
+    )
     (pin "1")
     (pin "2")
@@
     )
     (property "Tolerance" "1%" (id 6) (at 63.5 111.76 0)
+      (effects (font (size 1.27 1.27)) hide)
+    )
+    (property "DK" "13-RC0402FR-074M99LCT-ND" (id 7) (at 63.5 111.76 0)
       (effects (font (size 1.27 1.27)) hide)
     )
@@
       (effects (font (size 1.27 1.27)) hide)
     )
+    (property "DK" "490-GRM155D81C475ME15JCT-ND" (id 7) (at 119.38 106.68 0)
+      (effects (font (size 1.27 1.27)) hide)
+    )
